File: schema/RL2D/RL2D.kicad_sch (KiCad schematic)
At the start: 9 parts, among them J1 Steer_Joystick, SW1 SW_Brake, SW2 SW_Accel, SW3 SW_Superpower, SW4 SW_On, U1 ESP32_WROOM-32, U2 ILI9341

Commit message: progress 3/7
Parts:
- removed SW1: SW_Brake, symbol Switch:SW_Push
- removed SW2: SW_Accel, symbol Switch:SW_Push
- removed SW3: SW_Superpower, symbol Switch:SW_Push
- added SW1, SW2, SW3: SW_FancyButton, symbol RL2D:SW_FancyButton
- J1: footprint (none) -> RL2D:Joystick
- R1: renamed from R?; value R_US -> 330Ω
- U1: footprint (none) -> RL2D:ESP32
Connections:
- net +3V3: now also J1.1 (VCC), U1.1 (3V3); no longer J1.2 (VCC), U1. (VIN)
- net +9V: now also U1.29 (VIN); no longer U1. (VIN)
- net GND: now also J1.5 (GND), U1.2 (GND), SW1.2, SW2.2, SW3.1; no longer J1.1 (GND), U1. (VIN)
- net at J1.3 (Y): now also U1.28 (D13); no longer U1.12 (D12)
- net at J1.4 (S): now also U1.26 (D14); no longer U1.13 (D13)
- net at U1.14 (SCL): no longer J1.5 (SW)
- net at U2.4 (RESET): now also U1.4 (D2); no longer U1.2 (D2)
- net at U2.5 (D/~{C}): now also U1.5 (D4); no longer U1.4 (D4)
- net at U1.21 (D32): now also SW2.1
- net at U1.22 (D33): now also SW1.1
- net at U1.23 (D25): now also SW3.2
- net at U1.27 (D12): now also J1.2 (X)

Commit message: new esp32 schemas
Parts:
- removed U1: ESP32_WROOM-32, RL2D:ESP32, symbol RL2D:ESP32_WROOM-32
- removed U2: ILI9341, Display:CR2013-MI2120, symbol Driver_Display:CR2013-MI2120
- added MCU1: ESP32_WROOM-32, symbol RL2D:ESP32_WROOM-32
- added U1: ILI9341 2.8" TFT LCD, symbol RL2D:ILI9341 2.8{dblquote} TFT LCD
- BT1: value Battery -> 9V Battery
- R1: footprint (none) -> Resistor_THT:R_Axial_DIN0207_L6.3mm_D2.5mm_P10.16mm_Horizontal
- SW1, SW2, SW3: footprint (none) -> RL2D:FancyButton
- SW4: footprint (none) -> RL2D:Switch
Connections:
- net +3V3: now also MCU1.1 (3V3), U1.1 (VCC)
- net GND: now also SW1.1, SW2.1, MCU1.2 (GND), U1.2 (GND); no longer SW1.2, SW2.2
- net at J1.2 (X): now also MCU1.5 (D34)
- net at J1.3 (Y): now also MCU1.6 (D35)
- net at J1.4 (S): now also MCU1.7 (D32)
- net at R1.1: now also U1.8 (LED)
- net at SW3.2: now also MCU1.8 (D33)
- net +9V renamed VDC
- net VDC: now also MCU1.19 (VIN/5V)
- new net: MCU1.25 (D0), SW2.2
- new net: MCU1.26 (D4), SW1.2
- new net: MCU1.10 (D26), U1.4 (RESET)
- new net: MCU1.9 (D25), U1.5 (D/~{C})
Other:
- moved on the sheet: SW1, SW2

Commit message: pcbout
Parts:
- BT1: footprint (none) -> Connector_JST:JST_XH_B2B-XH-A_1x02_P2.50mm_Vertical
- MCU1: footprint (none) -> RL2D:ESP32
- U1: footprint (none) -> RL2D:ILI9341 2.8inch
Changed lines of the file:
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@@
   (symbol (lib_id "power:VDC") (at 35.56 100.33 90) (unit 1)
     (in_bom yes) (on_board yes) (fields_autoplaced)
-    (property "Reference" "#PWR?" (id 0) (at 38.1 100.33 0)
+    (property "Reference" "#PWR0113" (id 0) (at 38.1 100.33 0)
       (effects (font (size 1.27 1.27)) hide)
     )
@@
       (effects (font (size 1.27 1.27)) (justify left))
     )
-    (property "Footprint" "" (id 2) (at 161.29 71.12 0)
+    (property "Footprint" "RL2D:ESP32" (id 2) (at 161.29 71.12 0)
       (effects (font (size 1.27 1.27)) hide)
     )
@@
   (symbol (lib_id "power:VDC") (at 160.02 43.18 0) (unit 1)
     (in_bom yes) (on_board yes)
-    (property "Reference" "#PWR?" (id 0) (at 160.02 45.72 0)
+    (property "Reference" "#PWR0103" (id 0) (at 160.02 45.72 0)
       (effects (font (size 1.27 1.27)) hide)
     )
@@
       (effects (font (size 1.27 1.27)) (justify left))
     )
-    (property "Footprint" "" (id 2) (at 101.6 52.07 0)
+    (property "Footprint" "RL2D:ILI9341 2.8inch" (id 2) (at 101.6 52.07 0)
       (effects (font (size 1.27 1.27)) hide)
     )
@@
   (symbol (lib_id "power:+3V3") (at 162.56 43.18 0) (unit 1)
     (in_bom yes) (on_board yes)
-    (property "Reference" "#PWR?" (id 0) (at 162.56 46.99 0)
+    (property "Reference" "#PWR0104" (id 0) (at 162.56 46.99 0)
       (effects (font (size 1.27 1.27)) hide)
     )
@@
     (property "Reference" "BT1" (id 0) (at 40.259 92.71 90))
     (property "Value" "9V Battery" (id 1) (at 40.259 95.25 90))
-    (property "Footprint" "" (id 2) (at 39.116 100.33 90)
+    (property "Footprint" "Connector_JST:JST_XH_B2B-XH-A_1x02_P2.50mm_Vertical" (id 2) (at 39.116 100.33 90)
       (effects (font (size 1.27 1.27)) hide)
     )
@@
       (reference "#PWR0102") (unit 1) (value "GND") (footprint "")
     )
+    (path "/974c2d76-5b7f-45d4-a32a-7d0d8b0e4963"
+      (reference "#PWR0103") (unit 1) (value "VDC") (footprint "")
+    )
+    (path "/b965cb9e-8dec-46f9-8838-25676e9a9e1f"
+      (reference "#PWR0104") (unit 1) (value "+3V3") (footprint "")
+    )
     (path "/32a94fa4-9414-4f8e-a7b5-2450b6790f48"
       (reference "#PWR0105") (unit 1) (value "GND") (footprint "")
@@
     )
     (path "/577020f8-ca75-4017-b6c9-642bdab2ee0b"
-      (reference "#PWR?") (unit 1) (value "VDC") (footprint "")
-    )
-    (path "/974c2d76-5b7f-45d4-a32a-7d0d8b0e4963"
-      (reference "#PWR?") (unit 1) (value "VDC") (footprint "")
-    )
-    (path "/b965cb9e-8dec-46f9-8838-25676e9a9e1f"
-      (reference "#PWR?") (unit 1) (value "+3V3") (footprint "")
+      (reference "#PWR0113") (unit 1) (value "VDC") (footprint "")
     )
     (path "/fc74fec6-8899-4958-bb73-6ceed471866c"
-      (reference "BT1") (unit 1) (value "9V Battery") (footprint "")
+      (reference "BT1") (unit 1) (value "9V Battery") (footprint "Connector_JST:JST_XH_B2B-XH-A_1x02_P2.50mm_Vertical")
     )
     (path "/286ef0bb-63a2-4d30-a3f5-1f8488cb0b27"
@@
     )
     (path "/7a1fca65-8bdf-43b8-a702-3dfe016059c4"
-      (reference "MCU1") (unit 1) (value "ESP32_WROOM-32") (footprint "")
+      (reference "MCU1") (unit 1) (value "ESP32_WROOM-32") (footprint "RL2D:ESP32")
     )
     (path "/d85fdf4c-f3d7-4afa-83cb-40a0d4935c82"
@@
     )
     (path "/b7d46f5e-940d-4585-8638-f880da0f1ff6"
-      (reference "U1") (unit 1) (value "ILI9341 2.8\" TFT LCD") (footprint "")
-    )
-  )
+      (reference "U1") (unit 1) (value "ILI9341 2.8\" TFT LCD") (footprint "RL2D:ILI9341 2.8inch")
+    )
+  )

Commit message: progress 3/14
Parts:
- R1: footprint Resistor_THT:R_Axial_DIN0207_L6.3mm_D2.5mm_P10.16mm_Horizontal -> Resistor_THT:R_Axial_DIN0207_L6.3mm_D2.5mm_P15.24mm_Horizontal
Connections:
- net at MCU1.11 (D27): now also U1.3 (~{CS})
- net at MCU1.12 (SCK): now also U1.7 (SCK)
- net at MCU1.13 (MISO): now also U1.9 (MISO)
- net at MCU1.15 (MOSI): now also U1.6 (MOSI)
Other:
- moved on the sheet: R1
Changed lines of the file:
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@@
   (title_block
     (title "Rocket League 2D Main Schema")
-    (date "2024-03-09")
-    (rev "v0.6.1")
+    (date "2024-03-14")
+    (rev "v0.7")
     (company "Vrishak Vemuri (vninja007)")
   )
-  (bus_entry (at 123.19 34.29) (size 2.54 2.54)
-    (stroke (width 0) (type default) (color 0 0 0 0))
-  )
-  (bus_entry (at 147.32 74.93) (size 2.54 2.54)
-    (stroke (width 0) (type default) (color 0 0 0 0))
-  )
-  (bus_entry (at 147.32 82.55) (size 2.54 2.54)
-    (stroke (width 0) (type default) (color 0 0 0 0))
-  )
-  (bus_entry (at 147.32 72.39) (size 2.54 2.54)
-    (stroke (width 0) (type default) (color 0 0 0 0))
-  )
-  (bus_entry (at 123.19 36.83) (size 2.54 2.54)
-    (stroke (width 0) (type default) (color 0 0 0 0))
-  )
-  (bus_entry (at 123.19 29.21) (size 2.54 2.54)
-    (stroke (width 0) (type default) (color 0 0 0 0))
-  )
-  (bus_entry (at 123.19 31.75) (size 2.54 2.54)
-    (stroke (width 0) (type default) (color 0 0 0 0))
-  )
-  (bus_entry (at 147.32 77.47) (size 2.54 2.54)
-    (stroke (width 0) (type default) (color 0 0 0 0))
-  )
   (wire (pts (xy 123.19 39.37) (xy 123.19 40.64))
     (stroke (width 0) (type default) (color 0 0 0 0))
@@
     (stroke (width 0) (type default) (color 0 0 0 0))
   )
-  (wire (pts (xy 123.19 40.64) (xy 127 40.64))
+  (wire (pts (xy 123.19 40.64) (xy 133.35 40.64))
     (stroke (width 0) (type default) (color 0 0 0 0))
   )
@@
     (stroke (width 0) (type default) (color 0 0 0 0))
   )
-  (bus (pts (xy 125.73 31.75) (xy 125.73 34.29))
-    (stroke (width 0) (type default) (color 0 0 0 0))
-  )
   (wire (pts (xy 48.26 39.37) (xy 66.04 39.37))
     (stroke (width 0) (type default) (color 0 0 0 0))
@@
     (stroke (width 0) (type default) (color 0 0 0 0))
   )
+  (wire (pts (xy 121.92 34.29) (xy 129.54 34.29))
+    (stroke (width 0) (type default) (color 0 0 0 0))
+  )
   (wire (pts (xy 175.26 80.01) (xy 171.45 80.01))
     (stroke (width 0) (type default) (color 0 0 0 0))
   )
-  (bus (pts (xy 125.73 39.37) (xy 125.73 72.39))
-    (stroke (width 0) (type default) (color 0 0 0 0))
-  )
-  (bus (pts (xy 147.32 82.55) (xy 147.32 77.47))
-    (stroke (width 0) (type default) (color 0 0 0 0))
-  )
-  (wire (pts (xy 149.86 74.93) (xy 151.13 74.93))
+  (wire (pts (xy 129.54 34.29) (xy 129.54 80.01))
+    (stroke (width 0) (type default) (color 0 0 0 0))
+  )
+  (wire (pts (xy 132.08 74.93) (xy 151.13 74.93))
     (stroke (width 0) (type default) (color 0 0 0 0))
   )
@@
     (stroke (width 0) (type default) (color 0 0 0 0))
   )
-  (wire (pts (xy 134.62 26.67) (xy 134.62 38.1))
+  (wire (pts (xy 138.43 26.67) (xy 138.43 38.1))
     (stroke (width 0) (type default) (color 0 0 0 0))
   )
@@
     (stroke (width 0) (type default) (color 0 0 0 0))
   )
-  (wire (pts (xy 140.97 38.1) (xy 140.97 69.85))
+  (wire (pts (xy 144.78 38.1) (xy 144.78 69.85))
     (stroke (width 0) (type default) (color 0 0 0 0))
   )
@@
     (stroke (width 0) (type default) (color 0 0 0 0))
   )
-  (bus (pts (xy 147.32 74.93) (xy 147.32 72.39))
-    (stroke (width 0) (type default) (color 0 0 0 0))
-  )
-  (bus (pts (xy 125.73 36.83) (xy 125.73 39.37))
-    (stroke (width 0) (type default) (color 0 0 0 0))
-  )
   (wire (pts (xy 151.13 71.12) (xy 127 71.12))
     (stroke (width 0) (type default) (color 0 0 0 0))
   )
-  (wire (pts (xy 140.97 69.85) (xy 151.13 69.85))
+  (wire (pts (xy 144.78 69.85) (xy 151.13 69.85))
+    (stroke (width 0) (type default) (color 0 0 0 0))
+  )
+  (wire (pts (xy 128.27 31.75) (xy 128.27 85.09))
     (stroke (width 0) (type default) (color 0 0 0 0))
   )
@@
     (stroke (width 0) (type default) (color 0 0 0 0))
   )
-  (wire (pts (xy 121.92 29.21) (xy 123.19 29.21))
+  (wire (pts (xy 121.92 29.21) (xy 132.08 29.21))
     (stroke (width 0) (type default) (color 0 0 0 0))
   )
@@
     (stroke (width 0) (type default) (color 0 0 0 0))
   )
-  (wire (pts (xy 121.92 36.83) (xy 123.19 36.83))
-    (stroke (width 0) (type default) (color 0 0 0 0))
-  )
-  (wire (pts (xy 149.86 77.47) (xy 151.13 77.47))
+  (wire (pts (xy 132.08 29.21) (xy 132.08 74.93))
+    (stroke (width 0) (type default) (color 0 0 0 0))
+  )
+  (wire (pts (xy 130.81 77.47) (xy 151.13 77.47))
     (stroke (width 0) (type default) (color 0 0 0 0))
   )
@@
     (stroke (width 0) (type default) (color 0 0 0 0))
   )
-  (bus (pts (xy 125.73 34.29) (xy 125.73 36.83))
-    (stroke (width 0) (type default) (color 0 0 0 0))
-  )
-  (bus (pts (xy 147.32 72.39) (xy 125.73 72.39))
-    (stroke (width 0) (type default) (color 0 0 0 0))
-  )
-  (wire (pts (xy 149.86 80.01) (xy 151.13 80.01))
+  (wire (pts (xy 130.81 36.83) (xy 130.81 77.47))
+    (stroke (width 0) (type default) (color 0 0 0 0))
+  )
+  (wire (pts (xy 129.54 80.01) (xy 151.13 80.01))
     (stroke (width 0) (type default) (color 0 0 0 0))
   )
@@
     (stroke (width 0) (type default) (color 0 0 0 0))
   )
-  (wire (pts (xy 121.92 34.29) (xy 123.19 34.29))
-    (stroke (width 0) (type default) (color 0 0 0 0))
-  )
   (wire (pts (xy 175.26 38.1) (xy 175.26 80.01))
     (stroke (width 0) (type default) (color 0 0 0 0))
@@
     (stroke (width 0) (type default) (color 0 0 0 0))
   )
-  (wire (pts (xy 121.92 26.67) (xy 134.62 26.67))
-    (stroke (width 0) (type default) (color 0 0 0 0))
-  )
-  (bus (pts (xy 147.32 77.47) (xy 147.32 74.93))
-    (stroke (width 0) (type default) (color 0 0 0 0))
-  )
-  (wire (pts (xy 149.86 85.09) (xy 151.13 85.09))
-    (stroke (width 0) (type default) (color 0 0 0 0))
-  )
-  (wire (pts (xy 121.92 31.75) (xy 123.19 31.75))
-    (stroke (width 0) (type default) (color 0 0 0 0))
-  )
-  (wire (pts (xy 134.62 38.1) (xy 140.97 38.1))
+  (wire (pts (xy 121.92 26.67) (xy 138.43 26.67))
+    (stroke (width 0) (type default) (color 0 0 0 0))
+  )
+  (wire (pts (xy 128.27 85.09) (xy 151.13 85.09))
+    (stroke (width 0) (type default) (color 0 0 0 0))
+  )
+  (wire (pts (xy 121.92 31.75) (xy 128.27 31.75))
+    (stroke (width 0) (type default) (color 0 0 0 0))
+  )
+  (wire (pts (xy 121.92 36.83) (xy 130.81 36.83))
+    (stroke (width 0) (type default) (color 0 0 0 0))
+  )
+  (wire (pts (xy 138.43 38.1) (xy 144.78 38.1))
     (stroke (width 0) (type default) (color 0 0 0 0))
   )
@@
     (pin "1")
   )
-  (symbol (lib_id "power:+3V3") (at 134.62 40.64 270) (unit 1)
+  (symbol (lib_id "power:+3V3") (at 140.97 40.64 270) (unit 1)
     (in_bom yes) (on_board yes)
-    (property "Reference" "#PWR0101" (id 0) (at 130.81 40.64 0)
-      (effects (font (size 1.27 1.27)) hide)
-    )
-    (property "Value" "+3V3" (id 1) (at 135.89 43.18 90))
-    (property "Footprint" "" (id 2) (at 134.62 40.64 0)
-      (effects (font (size 1.27 1.27)) hide)
-    )
-    (property "Datasheet" "" (id 3) (at 134.62 40.64 0)
+    (property "Reference" "#PWR0101" (id 0) (at 137.16 40.64 0)
+      (effects (font (size 1.27 1.27)) hide)
+    )
+    (property "Value" "+3V3" (id 1) (at 142.24 43.18 90))
+    (property "Footprint" "" (id 2) (at 140.97 40.64 0)
+      (effects (font (size 1.27 1.27)) hide)
+    )
+    (property "Datasheet" "" (id 3) (at 140.97 40.64 0)
       (effects (font (size 1.27 1.27)) hide)
     )
@@
       (effects (font (size 1.27 1.27)) hide)
     )
-    (property "Value" "GND" (id 1) (at 139.7 34.29 90)
+    (property "Value" "GND" (id 1) (at 143.51 34.29 90)
       (effects (font (size 1.27 1.27)) (justify right))
     )
@@
     (pin "1")
   )
-  (symbol (lib_id "Device:R_US") (at 130.81 40.64 90) (unit 1)
-    (in_bom yes) (on_board yes) (fields_autoplaced)
-    (property "Reference" "R1" (id 0) (at 130.81 34.29 90))
-    (property "Value" "330Ω" (id 1) (at 130.81 36.83 90))
-    (property "Footprint" "Resistor_THT:R_Axial_DIN0207_L6.3mm_D2.5mm_P10.16mm_Horizontal" (id 2) (at 131.064 39.624 90)
-      (effects (font (size 1.27 1.27)) hide)
-    )
-    (property "Datasheet" "~" (id 3) (at 130.81 40.64 0)
+  (symbol (lib_id "Device:R_US") (at 137.16 40.64 90) (unit 1)
+    (in_bom yes) (on_board yes) (fields_autoplaced)
+    (property "Reference" "R1" (id 0) (at 137.16 34.29 90))
+    (property "Value" "330Ω" (id 1) (at 137.16 36.83 90))
+    (property "Footprint" "Resistor_THT:R_Axial_DIN0207_L6.3mm_D2.5mm_P15.24mm_Horizontal" (id 2) (at 137.414 39.624 90)
+      (effects (font (size 1.27 1.27)) hide)
+    )
+    (property "Datasheet" "~" (id 3) (at 137.16 40.64 0)
       (effects (font (size 1.27 1.27)) hide)
     )
@@
     )
     (path "/d85fdf4c-f3d7-4afa-83cb-40a0d4935c82"
-      (reference "R1") (unit 1) (value "330Ω") (footprint "Resistor_THT:R_Axial_DIN0207_L6.3mm_D2.5mm_P10.16mm_Horizontal")
+      (reference "R1") (unit 1) (value "330Ω") (footprint "Resistor_THT:R_Axial_DIN0207_L6.3mm_D2.5mm_P15.24mm_Horizontal")
     )
     (path "/51826c9c-7f94-482c-a534-f54edfec4ce1"
